Commit message: inverted z axis in CAD reference to match motion direction
Fingers parameters are based on try.

File: kinova_description/urdf/jaco2_arm.xacro (robot description, xacro)
@@ -34,7 +34,7 @@
   <property name="joint_base_origin_rpy" value="0 0 0" />
   <property name="joint_1" value="jaco2_joint_1" />
-  <property name="joint_1_axis_xyz" value="0 0 -1" />
+  <property name="joint_1_axis_xyz" value="0 0 1" />
   <property name="joint_1_origin_xyz" value="0 0 0.1535" />
-  <property name="joint_1_origin_rpy" value="${J_PI} 0 ${J_PI}" />
+  <property name="joint_1_origin_rpy" value="0 ${J_PI} 0" />
   <property name="joint_1_lower_limit" value="${-2*J_PI}" />
   <property name="joint_1_upper_limit" value="${2*J_PI}" />
@@ -42,40 +42,41 @@
   <property name="joint_2_axis_xyz" value="0 0 1" />
   <property name="joint_2_origin_xyz" value="0 0 -0.1185" />
-  <property name="joint_2_origin_rpy" value="-${J_PI/2} ${J_PI} 0" />
+  <property name="joint_2_origin_rpy" value="${-J_PI/2} 0 ${J_PI}" />
   <property name="joint_2_lower_limit" value="${-J_PI}" />
   <property name="joint_2_upper_limit" value="${0}" />
   <property name="joint_3" value="jaco2_joint_3" />
-  <property name="joint_3_axis_xyz" value="0 0 -1" />
-  <property name="joint_3_origin_xyz" value="0.41 0 0" />
-  <property name="joint_3_origin_rpy" value="${J_PI} 0 ${J_PI/2}" />
+  <property name="joint_3_axis_xyz" value="0 0 1" />
+  <property name="joint_3_origin_xyz" value="0 -0.41 0" />
+  <property name="joint_3_origin_rpy" value="${J_PI} 0 ${J_PI}" />
   <property name="joint_3_lower_limit" value="${-5*J_PI/4}" />
   <property name="joint_3_upper_limit" value="${1*J_PI/4}" />
   <property name="joint_4" value="jaco2_joint_4" />
-  <property name="joint_4_axis_xyz" value="0 0 -1" />
-  <property name="joint_4_origin_xyz" value="0.207 0 -0.01125" />
-  <property name="joint_4_origin_rpy" value="${J_PI} ${J_PI/2} 0" />
+  <property name="joint_4_axis_xyz" value="0 0 1" />
+  <property name="joint_4_origin_xyz" value="0 0.207 -0.01125" />
+  <property name="joint_4_origin_rpy" value="${J_PI/2} 0 0" />
   <property name="joint_4_lower_limit" value="${-2*J_PI}" />
   <property name="joint_4_upper_limit" value="${2*J_PI}" />
   <property name="joint_5" value="jaco2_joint_5" />
-  <property name="joint_5_axis_xyz" value="0 0 -1" />
-  <property name="joint_5_origin_xyz" value="0.03700 0 -0.06408" />
-  <property name="joint_5_origin_rpy" value="0 -${J_PI/180*60} 0" />
+  <property name="joint_5_axis_xyz" value="0 0 1" />
+  <property name="joint_5_origin_xyz" value="0 -0.03700 -0.06408" />
+  <property name="joint_5_origin_rpy" value="${J_PI/3} 0 ${J_PI}" />
   <property name="joint_5_lower_limit" value="${-2*J_PI}" />
   <property name="joint_5_upper_limit" value="${2*J_PI}" />
   <property name="joint_6" value="jaco2_joint_6" />
-  <property name="joint_6_axis_xyz" value="0 0 -1" />
-  <property name="joint_6_origin_xyz" value="0.03700 0 -0.06408" />
-  <property name="joint_6_origin_rpy" value="-${J_PI/180*60} 0 ${J_PI/2}" />
+  <property name="joint_6_axis_xyz" value="0 0 1" />
+  <property name="joint_6_origin_xyz" value="0 -0.03700 -0.06408" />
+  <property name="joint_6_origin_rpy" value="${-J_PI/3} 0 0" />
   <property name="joint_6_lower_limit" value="${-2*J_PI}" />
   <property name="joint_6_upper_limit" value="${2*J_PI}" />
   <property name="joint_finger_1" value="jaco2_joint_finger_1" />
   <property name="joint_finger_1_axis_xyz" value="0 0 1" />
-  <property name="joint_finger_1_origin_xyz" value="-0.03978 0 -0.10071" />
-  <property name="joint_finger_1_origin_rpy" value="-1.7983 1.117 3.1416" />
+  <property name="joint_finger_1_origin_xyz" value="0 0.032 -0.114" />
+  <!-- <property name="joint_finger_1_origin_rpy" value="-1.7983 1.117 3.1416" /> -->
+  <property name="joint_finger_1_origin_rpy" value="0 ${J_PI/2} ${J_PI}" />
   <property name="joint_finger_1_lower_limit" value="0" />
   <property name="joint_finger_1_upper_limit" value="${J_PI/180*40}" />
   <property name="joint_finger_tip_1" value="jaco2_joint_finger_tip_1" />
   <property name="joint_finger_tip_1_axis_xyz" value="0 0 1" />
-  <property name="joint_finger_tip_1_origin_xyz" value="0.035 -0.02595 -0.0025" />
+  <property name="joint_finger_tip_1_origin_xyz" value="0.042 -0.00595 -0.0025" />
   <property name="joint_finger_tip_1_origin_rpy" value="0 0 0" />
   <property name="joint_finger_tip_1_lower_limit" value="0" />
@@ -86,11 +87,11 @@
   <property name="joint_finger_2" value="jaco2_joint_finger_2" />
   <property name="joint_finger_2_axis_xyz" value="0 0 1" />
-  <property name="joint_finger_2_origin_xyz" value="0.03569 -0.0216 -0.10071" />
-  <property name="joint_finger_2_origin_rpy" value="-1.6222 1.117 -0.23615" />
+  <property name="joint_finger_2_origin_xyz" value="-0.025 -0.0256 -0.105" />
+  <property name="joint_finger_2_origin_rpy" value="0 ${J_PI/2} 0" />
   <property name="joint_finger_2_lower_limit" value="0" />
   <property name="joint_finger_2_upper_limit" value="${J_PI/180*40}" />
   <property name="joint_finger_tip_2" value="jaco2_joint_finger_tip_2" />
   <property name="joint_finger_tip_2_axis_xyz" value="0 0 1" />
-  <property name="joint_finger_tip_2_origin_xyz" value="0.035 -0.02595 -0.0025" />
+  <property name="joint_finger_tip_2_origin_xyz" value="0.045 -0.00595 -0.0025" />
   <property name="joint_finger_tip_2_origin_rpy" value="0 0 0" />
   <property name="joint_finger_tip_2_lower_limit" value="0" />
@@ -101,11 +102,11 @@
   <property name="joint_finger_3" value="jaco2_joint_finger_3" />
   <property name="joint_finger_3_axis_xyz" value="0 0 1" />
-  <property name="joint_finger_3_origin_xyz" value="0.03569 0.0216 -0.10071" />
-  <property name="joint_finger_3_origin_rpy" value="-1.5161 1.1459 0.23978" />
+  <property name="joint_finger_3_origin_xyz" value="0.025 -0.0256 -0.105" />
+  <property name="joint_finger_3_origin_rpy" value="0 ${J_PI/2} 0" />
   <property name="joint_finger_3_lower_limit" value="0" />
   <property name="joint_finger_3_upper_limit" value="${J_PI/180*40}" />
   <property name="joint_finger_tip_3" value="jaco3_joint_finger_tip_3" />
   <property name="joint_finger_tip_3_axis_xyz" value="0 0 1" />
-  <property name="joint_finger_tip_3_origin_xyz" value="0.035 -0.02595 -0.0025" />
+  <property name="joint_finger_tip_3_origin_xyz" value="0.045 -0.00595 -0.0025" />
   <property name="joint_finger_tip_3_origin_rpy" value="0 0 0" />
   <property name="joint_finger_tip_3_lower_limit" value="0" />

File: kinova_description/urdf/standalone_jaco2.xacro.urdf (robot description, URDF)
Before this commit: robot jaco, 16 links, 15 joints
Links:
- removed link finger_distal_limb_1
- removed link finger_distal_limb_2
- removed link finger_distal_limb_3
- removed link finger_proximal_limb_1
- removed link finger_proximal_limb_2
- removed link finger_proximal_limb_3
- added link jaco2_link_finger_1; collision mesh filename=package://kinova_description/meshes/jaco2_link_finger_1.dae; visual mesh filename=package://kinova_description/meshes/jaco2_link_finger_1.dae
- added link jaco2_link_finger_2; collision mesh filename=package://kinova_description/meshes/jaco2_link_finger_2.dae; visual mesh filename=package://kinova_description/meshes/jaco2_link_finger_2.dae
- added link jaco2_link_finger_3; collision mesh filename=package://kinova_description/meshes/jaco2_link_finger_3.dae; visual mesh filename=package://kinova_description/meshes/jaco2_link_finger_3.dae
- added link jaco2_link_finger_tip_1; collision mesh filename=package://kinova_description/meshes/jaco2_link_finger_tip_1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; visual mesh filename=package://kinova_description/meshes/jaco2_link_finger_tip_1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
- added link jaco2_link_finger_tip_2; collision mesh filename=package://kinova_description/meshes/jaco2_link_finger_tip_2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; visual mesh filename=package://kinova_description/meshes/jaco2_link_finger_tip_2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
- added link jaco2_link_finger_tip_3; collision mesh filename=package://kinova_description/meshes/jaco2_link_finger_tip_3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; visual mesh filename=package://kinova_description/meshes/jaco2_link_finger_tip_3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
- link jaco2_link_1: geometry collision mesh filename=package://kinova_description/meshes/jaco2_link_1.dae; visual mesh filename=package://kinova_description/meshes/jaco2_link_1.dae
- link jaco2_link_2: geometry collision mesh filename=package://kinova_description/meshes/jaco2_link_2.dae; visual mesh filename=package://kinova_description/meshes/jaco2_link_2.dae
- link jaco2_link_3: geometry collision mesh filename=package://kinova_description/meshes/jaco2_link_3.dae; visual mesh filename=package://kinova_description/meshes/jaco2_link_3.dae
- link jaco2_link_4: geometry collision mesh filename=package://kinova_description/meshes/jaco2_link_4.dae; visual mesh filename=package://kinova_description/meshes/jaco2_link_4.dae
- link jaco2_link_5: geometry collision mesh filename=package://kinova_description/meshes/jaco2_link_5.dae; visual mesh filename=package://kinova_description/meshes/jaco2_link_5.dae
- link jaco2_link_base: geometry collision mesh filename=package://kinova_description/meshes/jaco2_link_base.dae; visual mesh filename=package://kinova_description/meshes/jaco2_link_base.dae
- link jaco2_link_hand: geometry collision mesh filename=package://kinova_description/meshes/jaco2_link_hand.dae; visual mesh filename=package://kinova_description/meshes/jaco2_link_hand.dae
Joints:
- joint jaco2_joint_1: origin xyz=0 0 0.1535 rpy=3.14159265359 0 3.14159265359 -> xyz=0 0 0.1535 rpy=0 0 0
- joint jaco2_joint_2: origin xyz=0 0 -0.1185 rpy=-1.57079632679 3.14159265359 0 -> xyz=0 0 0.1185 rpy=1.57079632679 0 0
- joint jaco2_joint_finger_1: child finger_proximal_limb_1 -> jaco2_link_finger_1
- joint jaco2_joint_finger_2: child finger_proximal_limb_2 -> jaco2_link_finger_2
- joint jaco2_joint_finger_3: child finger_proximal_limb_3 -> jaco2_link_finger_3
- joint jaco2_joint_finger_tip_1: child finger_distal_limb_1 -> jaco2_link_finger_tip_1; parent finger_proximal_limb_1 -> jaco2_link_finger_1
- joint jaco2_joint_finger_tip_2: child finger_distal_limb_2 -> jaco2_link_finger_tip_2; parent finger_proximal_limb_2 -> jaco2_link_finger_2
- joint jaco3_joint_finger_tip_3: child finger_distal_limb_3 -> jaco2_link_finger_tip_3; parent finger_proximal_limb_3 -> jaco2_link_finger_3
