Commit message: fix mimic in URDF model

File: kinova_description/urdf/kinova_common.xacro (robot description, xacro)
@@ -75,5 +75,5 @@
         </joint>
         <xacro:kinova_armlink link_name="${prefix}_link_finger_tip_${finger_number}" link_mesh="finger_distal"/>
-        <joint name="${prefix}_joint_finger_tip_${finger_number}" type="fixed">
+        <joint name="${prefix}_joint_finger_tip_${finger_number}" type="revolute">
             <parent link="${prefix}_link_finger_${finger_number}"/>
             <child link="${prefix}_link_finger_tip_${finger_number}"/>
@@ -81,5 +81,5 @@
             <origin xyz="0.044 -0.003 0" rpy="0 0 0"/>
             <limit lower="0" upper="2" effort="30" velocity="5"/>
-            <mimic joint="${J_PI/180*40}" multiplier="1.0" offset="0.0"/>
+            <mimic joint="${prefix}_joint_finger_${finger_number}" multiplier="0.5"/>
         </joint>
     </xacro:macro>

Commit message: reduce mimic joint value of finger tip

File: kinova_description/urdf/kinova_common.xacro (robot description, xacro)
@@ -81,5 +81,5 @@
             <origin xyz="0.044 -0.003 0" rpy="0 0 0"/>
             <limit lower="0" upper="2" effort="30" velocity="5"/>
-            <mimic joint="${prefix}_joint_finger_${finger_number}" multiplier="0.5"/>
+            <mimic joint="${prefix}_joint_finger_${finger_number}" multiplier="0.1"/>
         </joint>
     </xacro:macro>
